File: FSCS.kicad_pcb (KiCad board)
At the start: 2 copper layers, 65.9 x 62.4 mm, 66 parts, among them J1 BMP280, J10 GPS, J11 Conn_01x03_Pin, J12 Conn_01x02_Pin, J13 Conn_01x02_Pin, J2 Conn_01x03_Pin, J3 Conn_01x03_Pin, J4 Conn_01x08_Pin, J5 Conn_01x20_Pin, J6 Conn_01x08_Pin, J7 USB_C_Receptacle_USB2.0_16P, J8 Conn_01x03_Pin, J9 Conn_01x03_Pin, U1 NCP1117-3.3_SOT223, U2 RP2350B-QFN80, U3 W25Q128JVSIQ TR, U4 MPU-6050, X1 ABM8-272-T3

Commit message: Update all project files
Parts:
- removed the G*** at (154.0, 110.3)

Commit message: Update plot files
Other:
- board text removed: "TANISHQ"
Changed lines of the file:
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@@
-		)
-	)
-	(gr_text "TANISHQ"
-		(at 145.19 121.15 0)
-		(layer "B.SilkS")
-		(effects
-			(font
-				(size 4 4)
-				(thickness 1)
-				(bold yes)
-			)
-			(justify left bottom mirror)
 		)
 	)
