File: FSCS.kicad_sch (KiCad schematic)
At the start: 0 parts

Commit message: schematic
Other:
- note removed: "camera to be added at last"
- note removed: "peripherals like mpu6050 and others to be done later"
- note removed: "pin connection for rp_usb and esp_usb to be done later"
- note removed: "the communication protocol between the 2 mcu to be decided before peripherals"
Changed lines of the file:
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@@
 	(generator_version "9.0")
 	(paper "A4")
-	(text "pin connection for rp_usb and esp_usb\nto be done later\n"
-		(exclude_from_sim no)
-		(at 146.812 49.53 0)
-		(effects
-			(font
-				(size 1.27 1.27)
-			)
-		)
-	)
-	(text "camera to be added at last\n"
-		(exclude_from_sim no)
-		(at 144.78 79.756 0)
-		(effects
-			(font
-				(size 1.27 1.27)
-			)
-		)
-	)
-	(text "the communication protocol between the 2 mcu to be decided before peripherals\n"
-		(exclude_from_sim no)
-		(at 153.162 89.154 0)
-		(effects
-			(font
-				(size 1.27 1.27)
-			)
-		)
-	)
-	(text "peripherals like mpu6050 and others to be done later\n"
-		(exclude_from_sim no)
-		(at 148.336 66.294 0)
-		(effects
-			(font
-				(size 1.27 1.27)
-			)
-		)
-	)
 	(sheet
 		(at 38.1 66.04)
@@
 	)
 	(sheet
-		(at 38.1 40.64)
+		(at 38.1 54.61)
 		(size 12.7 3.81)
 		(exclude_from_sim no)
@@
 		)
 		(property "Sheetname" "POWER"
-			(at 38.1 39.9284 0)
+			(at 38.1 53.8984 0)
 			(effects
 				(font
@@
 		)
 		(property "Sheetfile" "POWER.kicad_sch"
-			(at 38.1 45.0346 0)
+			(at 38.1 59.0046 0)
 			(effects
 				(font
